File: PCB/cadProd_compact.kicad_pcb (KiCad board)
At the start: 4 copper layers, 71 x 42.8 mm, 76 parts, among them J1 USB_B_Micro, J2 USB_Through_hole

Commit message: sum sum
Parts:
- removed +REG, BAT, USB+: TestPoint_Pad_1.0x1.0mm, TestPoint:TestPoint_Pad_1.0x1.0mm
- removed DigVol1: MCP1825S-1802E_DB, MCP1825S-1802E_DB:SOT230P700X180-4N
- added C19: 100nF, Capacitor_SMD:C_0805_2012Metric_Pad1.18x1.45mm_HandSolder, F.Cu at (175.2, 91.9)
- added C20: 10uF, Capacitor_SMD:C_0805_2012Metric_Pad1.18x1.45mm_HandSolder, F.Cu at (177.2, 91.9)
- added C21: 10uF, Capacitor_SMD:C_0805_2012Metric_Pad1.18x1.45mm_HandSolder, F.Cu at (186.7, 93.3)
- added C22: 100nF, Capacitor_SMD:C_0805_2012Metric_Pad1.18x1.45mm_HandSolder, F.Cu at (184.7, 93.3)
- added C23: 47nF, Capacitor_SMD:C_0805_2012Metric_Pad1.18x1.45mm_HandSolder, F.Cu at (181.8, 97.3)
- added C25: 100nF, Capacitor_SMD:C_0805_2012Metric_Pad1.18x1.45mm_HandSolder, F.Cu at (164.4, 88.4)
- added Digital_Vol1: TPS7A2033, Package_TO_SOT_SMD:SOT-23-5, F.Cu at (185.4, 98.3)
- added Q2: AO3401A, Package_TO_SOT_SMD:SOT-23, F.Cu at (180.2, 91.2)
- added R25: 100kOhm, Resistor_SMD:R_0805_2012Metric_Pad1.20x1.40mm_HandSolder, F.Cu at (181.8, 95.3)
- added R26: 10kOhm, Resistor_SMD:R_0805_2012Metric_Pad1.20x1.40mm_HandSolder, F.Cu at (178.8, 96.3)
- added R27: 1MOhm, Resistor_SMD:R_0805_2012Metric_Pad1.20x1.40mm_HandSolder, F.Cu at (162.0, 92.4)
- Battery1: footprint Crystal:Resonator-2Pin_W6.0mm_H3.0mm -> Connector_JST:JST_PH_B2B-PH-K_1x02_P2.00mm_Vertical
- R19, R20: value 10kOhm -> 20kOhm +
- R23, R24: value 10kOhm -> 3.9kOhm
- R5: value 10kOhm -> 1MOhm
- moved R5 16.3 mm to (160.0, 92.4), turned to 90 degrees
- moved A3v3 10.3 mm to (202.3, 97.7)
- moved R16 10.3 mm to (192.4, 99.7)
- moved AnaVol1 10.3 mm to (197.1, 98.7)
- moved REF** 6.50 mm to (192.5, 65.0)
- moved Battery1 4.40 mm to (160.6, 98.8), turned to 90 degrees
- moved R12 4.40 mm to (189.7, 89.8)
- moved BOOT1 4.30 mm to (190.7, 93.5)
- moved R7 2.97 mm to (163.0, 75.9)
- moved AUX1 2.92 mm to (204.2, 69.8), turned to 180 degrees
- moved C1 2.75 mm to (162.0, 79.5)
- moved C2 2.75 mm to (164.0, 79.5)
- moved R6 2.63 mm to (162.8, 83.0)
Connections:
- BATPROT1 pad 5: D3v3 -> AwO_D3v3
- Battery1 pad 1: BAT+ -> GND
- Battery1 pad 2: GND -> BAT+
- C6 pad 1: D3v3 -> AwO_D3v3
- C7 pad 1: D3v3 -> AwO_D3v3
- C8 pad 1: D3v3 -> AwO_D3v3
- ESP1 pad 2: D3v3 -> AwO_D3v3
- R10 pad 2: D3v3 -> AwO_D3v3
- R11 pad 2: D3v3 -> AwO_D3v3
- R12 pad 2: D3v3 -> AwO_D3v3
- R5 pad 1: D3v3 -> BAT+
- R5 pad 2: Det -> GPIO
- R9 pad 2: D3v3 -> AwO_D3v3
Routing:
- net AmpL: track 20.2 -> 32.0 mm
- net AwO_D3v3: track 0.00 -> 10.4 mm, vias 0 -> 5
- net EN_ANAVOL: track 18.0 -> 7.84 mm
- net D3v3: track 18.5 -> 10.2 mm, vias 12 -> 4
- net AmpR: track 28.7 -> 23.4 mm
- net USB+: track 39.5 -> 44.5 mm
- net DAT3SD: track 18.8 -> 14.0 mm
- net CMDSD: track 18.4 -> 13.7 mm
- net BAT+: track 2.35 -> 0.00 mm
- net BOOT: track 5.50 -> 7.75 mm
- net DAT0SD: track 12.9 -> 11.4 mm
- net +REG: track 1.30 -> 0.00 mm
- net D+: track 26.2 -> 27.1 mm
- net GND: track 87.0 -> 87.9 mm, vias 85 -> 66
- net D-: track 24.4 -> 25.1 mm
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- removed copper zone on F.Cu, net +REG
