File: PCB/cadProd_compact.kicad_sch (KiCad schematic)
At the start: 73 parts, among them J1 USB_B_Micro, J2 USB_Through_hole

Commit message: sum sum
Parts:
- removed DigVol1: MCP1825S-1802E_DB, MCP1825S-1802E_DB:SOT230P700X180-4N, symbol MCP1825S-1802E_DB:MCP1825S-1802E_DB
- removed ESD1, ESD2: PESD5V0L1BA1, Diode_SMD:D_SOD-323, symbol Diode:RF01VM2S
- removed R1, R2: 5.1kOhm, Resistor_SMD:R_0805_2012Metric_Pad1.20x1.40mm_HandSolder, symbol Device:R
- removed USBC1: USB_C_Receptacle_USB2.0_16P, Connector_USB:USB_C_Receptacle_GCT_USB4105-xx-A_16P_TopMnt_Horizontal, symbol Connector:USB_C_Receptacle_USB2.0_16P
- added C19, C22, C25: 100nF, Capacitor_SMD:C_0805_2012Metric_Pad1.18x1.45mm_HandSolder, symbol Device:C
- added C20, C21: 10uF, Capacitor_SMD:C_0805_2012Metric_Pad1.18x1.45mm_HandSolder, symbol Device:C
- added C23: 47nF, Capacitor_SMD:C_0805_2012Metric_Pad1.18x1.45mm_HandSolder, symbol Device:C
- added Digital_Vol1: TPS7A2033, Package_TO_SOT_SMD:SOT-23-5, symbol Regulator_Linear:AP2112K-3.3
- added Q2: AO3401A, Package_TO_SOT_SMD:SOT-23, symbol Transistor_FET:AO3401A
- added R25: 100kOhm, Resistor_SMD:R_0805_2012Metric_Pad1.20x1.40mm_HandSolder, symbol Device:R
- added R26: 10kOhm, Resistor_SMD:R_0805_2012Metric_Pad1.20x1.40mm_HandSolder, symbol Device:R
- added R27: 1MOhm, Resistor_SMD:R_0805_2012Metric_Pad1.20x1.40mm_HandSolder, symbol Device:R
- Battery1: footprint Crystal:Resonator-2Pin_W6.0mm_H3.0mm -> Connector_JST:JST_PH_B2B-PH-K_1x02_P2.00mm_Vertical
- R23, R24: value 10kOhm -> 3.9kOhm
- R5: value 10kOhm -> 1MOhm
Connections:
- net +REG: now also Digital_Vol1.1 (VIN), Digital_Vol1.3 (EN)
- net BAT+: now also Battery1.2 (+), R5.1; no longer Battery1.1 (+)
- net D3v3: now also C19.2, C20.2, Q2.3 (D); no longer BATPROT1.5 (EN2), C6.1, C7.1, C8.1, ESP1.2 (3V3), R10.2, R11.2, R12.2, R5.1, R9.2
- net Det: no longer R5.2
- net GND: now also Battery1.1 (-), C19.1, C20.1, C21.1, C22.1, C25.2, Digital_Vol1.2 (GND), R27.2; no longer Battery1.2 (-)
- new net: C23.2, Q2.1 (G), R25.2, R26.1
- new net AwO_D3v3: BATPROT1.5 (EN2), C21.2, C22.2, C23.1, C6.1, C7.1, C8.1, Digital_Vol1.5 (VOUT), ESP1.2 (3V3), Q2.2 (S), R10.2, R11.2, R12.2, R25.1, R9.2
- new net GPIO: C25.1, R26.2, R27.1, R5.2
- no-connect marks 8 -> 6
Other:
- moved on the sheet: Battery1
